File: 4 bit Full Adder 74HC.kicad_pcb (KiCad board)
At the start: 2 copper layers, 100 x 100 mm, 35 parts, among them J1 Screw_Terminal_01x02, J2 Screw_Terminal_01x02, SW1 SW_DIP_x04, SW2 SW_DIP_x04, SW3 SW_DIP_x01, U1 74HC86, U2 74HC86, U3 74LS08, U4 LM7805_TO220, U5 74LS32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

Commit message: Github
Parts:
- added G***: LOGO, Logos:spark_logo_wireframe, F.Cu at (251.5, 62.5)
