File: 4 bit Full Adder 74HC.kicad_sch (KiCad schematic)
At the start: 35 parts, among them J1 Screw_Terminal_01x02, J2 Screw_Terminal_01x02, SW1 SW_DIP_x04, SW2 SW_DIP_x04, SW3 SW_DIP_x01, U1 74HC86, U2 74HC86, U3 74LS08, U4 LM7805_TO220, U5 74LS32, U6 74LS08

Commit message: Update PCB, project file and Schematic
Other:
- company: Spark International -> (none)
Changed lines of the file:
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@@
 	(title_block
 		(title "4-bit Input Full Adder 74HC/LS")
-		(company "Spark International")
 		(comment 1 "Author: lion1113")
-		(comment 2 "6c623133")
-		(comment 3 "=)")
 	)
 	(junction
